File: pcb/resoncance_converter_controller/analog.kicad_sch (KiCad schematic)
At the start: 45 parts, among them U10 INA280A1xDCK, U11 INA280A1xDCK, U12 INA280A1xDCK, U17 TL3116, U5 OPA2325, U7 OPA2356xxDGK, U8 OPA356xxDBV, U9 INA280A1xDCK

Commit message: Finish first schematic resivion of the SOM
Parts:
- removed R30: 10K, Resistor_SMD:R_0402_1005Metric, symbol Device:R
- added C87, C88, C89: 100nF, Capacitor_SMD:C_0402_1005Metric, symbol Device:C
- added D24: ESD9B3.3ST5G, Diode_SMD:D_SOD-923, symbol Diode:ESD9B3.3ST5G
- added R60, R62, R65, R66: 10K, Resistor_SMD:R_0402_1005Metric, symbol Device:R
- added R61: 20K, Resistor_SMD:R_0402_1005Metric, symbol Device:R
- added R63, R64: 100K, Resistor_SMD:R_0402_1005Metric, symbol Device:R
- added RV1: 20K, Potentiometer_SMD:Potentiometer_Bourns_3269W_Vertical, symbol Device:R_Potentiometer
- added U18: OPA2356xxDGK, Package_SO:SOIC-8_3.9x4.9mm_P1.27mm, symbol Amplifier_Operational:OPA2356xxDGK
- added U19: OPA2325, Package_SO:SOIC-8_3.9x4.9mm_P1.27mm, symbol Amplifier_Operational:OPA2325
- added U20: OPA356xxDBV, Package_TO_SOT_SMD:SOT-23-5, symbol Amplifier_Operational:OPA356xxDBV
Connections:
- net +3.3V: now also C87.2, C88.2, C89.2, U18.8 (V+), U19.8 (V+), U20.5 (V+)
- net GND: now also C87.1, C88.1, C89.1, D24.1 (A1), R65.1, RV1.1, U18.3 (+), U18.4 (V-), U19.4 (V-), U20.2 (V-)
- net at R29.2, U5.2 (-): now also RV1.2, RV1.3
- new net: R60.2, R62.1, U18.2 (-)
- new net: R62.2, R63.2, U18.1
- new net: R61.2, U18.5 (+)
- new net: R64.1, U18.6 (-), U18.7
- new net: R65.2, R66.1, U20.4 (-)
- new net: R63.1, R64.2, U20.3 (+)
- new net FB_OCD2: D24.2 (A2), R60.1, R61.1
- new net FB_OCD2_RECTIFIED: R66.2, U20.1
