File: pcb/resoncance_converter_controller/controller.kicad_sch (KiCad schematic)
At the start: 25 parts, among them J1 Micro_SD_Card_Det2, U13 STM32G474VEHx, U14 APS6404L-SQRx-ZR, U15 APS6404L-SQRx-ZR, U16 AT24CS32-XHM, Y1 16Mhz

Commit message: Finish first schematic resivion of the SOM
Parts:
- added C90, C92, C93: 100nF, Capacitor_SMD:C_0402_1005Metric, symbol Device:C
- added C91: 10uF, Capacitor_SMD:C_2220_5750Metric, symbol Device:C
- added R67: 0R, Resistor_SMD:R_0402_1005Metric, symbol Device:R
- added R68: 240K, Resistor_SMD:R_0402_1005Metric, symbol Device:R
- added R69: 100K, Resistor_SMD:R_0402_1005Metric, symbol Device:R
- added U21: TPS2553DRVR, TPS2553DRVR:SON65P200X200X80-7N, symbol TPS2553DRVR:TPS2553DRVR
- C84: value 100nF -> 100uF; footprint Capacitor_SMD:C_0805_2012Metric -> Capacitor_SMD:C_2220_5750Metric
Connections:
- net +3.3V: now also R67.1, R69.2; no longer C84.1, J1.4 (VDD), R39.1, R40.2
- net CTRL_RX: now also U13.B3 (PE1); no longer U13.J3 (PC5)
- net CTRL_TX: now also U13.C4 (PE0); no longer U13.K2 (PC4)
- net GND: now also C90.2, C91.2, C92.2, C93.2, R68.2, U21.5 (GND), U21.7 (EP)
- net ISENSE1: now also U13.H3 (PA3); no longer U13.K3 (PB1)
- net ISENSE2: now also U13.G5 (PE7); no longer U13.H3 (PA3)
- net ISENSE3: now also U13.K3 (PB1); no longer U13.F4 (PC1)
- net ISENSE4: now also U13.F4 (PC1); no longer U13.G5 (PE7)
- net LCD_BL: now also U13.B8 (PD0); no longer U13.H5 (PE8)
- net LCD_DC: now also U13.A9 (PD1); no longer U13.H6 (PE9)
- net LCD_MISO: now also U13.C7 (PC11); no longer U13.B1 (PE5)
- net LCD_MOSI: now also U13.A10 (PC12); no longer U13.C2 (PE6)
- net LCD_RST: now also U13.B7 (PD2); no longer U13.K6 (PE10)
- net LCD_SCK: now also U13.C8 (PC10); no longer U13.C3 (PE2)
- net LCD_SS: now also U13.B9 (PA15); no longer U13.A1 (PE4)
- net QSPI_BK2_IO1: now also U13.F1 (PC2); no longer U13.A7 (PD5)
- net QSPI_BK2_IO2: now also U13.G1 (PC3); no longer U13.A6 (PD6)
- net QSPI_NCS: now also U13.C6 (PD3); no longer U13.H1 (PA2)
- net SD_CARD_DETECT: now also U13.B4 (PB7)
- net SD_MISO: now also U13.C2 (PE6); no longer U13.C7 (PC11)
- net SD_MOSI: now also U13.B1 (PE5); no longer U13.A10 (PC12)
- net SD_SCK: now also U13.C3 (PE2); no longer U13.C8 (PC10)
- net SD_SS: now also U13.A1 (PE4); no longer U13.B9 (PA15)
- net VSENSE: now also U13.H1 (PA2); no longer U13.J10 (PD12)
- net HRTIM_EEV9: now reaches U13.A5 (PB3)
- net ENCODER_CHB: now reaches U13.B2 (PE3)
- net POWER_INT: now reaches U13.C1 (PC14)
- net VOUT_ENABLE: now reaches U13.D1 (PC15)
- net GPIO3: now reaches U13.G10 (PD15)
- net AUX_PWM_CH2: now reaches U13.G2 (PA1)
- net AUX_PWM_CH1: now reaches U13.G4 (PA0)
- net GPIO0: now reaches U13.G7 (PD10)
- net GPIO1: now reaches U13.G8 (PD9)
- net GPIO2: now reaches U13.G9 (PD13)
- net FAN_PWM: now reaches U13.J2 (PA6)
- net ENCODER_CHA: now reaches U13.J4 (PB2)
- net GPIO6: now reaches U13.J6 (PE11)
- net HRTIM_FLT3: now reaches U13.J8 (PB10)
- new net: C84.1, C91.1, C92.1, J1.4 (VDD), R39.1, R40.2, U21.1 (OUT)
- new net: C90.1, U21.6 (IN)
- new net: R67.2, R68.1, U21.2 (ILIM)
- new net: C93.1, R69.1, U21.3 (~{FAULT}), U21.4 (EN)
- new net AUX_RX: U13.A6 (PD6)
- new net AUX_TX: U13.A7 (PD5)
- new net FB_OCD2: U13.J10 (PD12)
- new net GPIO4: U13.H5 (PE8)
- new net GPIO5: U13.H6 (PE9)
- new net GPIO7: U13.K6 (PE10)
Other:
- note added: "3.3 bus max 100mA"
- moved on the sheet: J1, R39, R40
