File: pcb/resoncance_converter_controller/resoncance_converter_controller.kicad_pcb (KiCad board)
At the start: 2 copper layers, 209 parts, among them J1 Micro_SD_Card_Det2, J10 Conn_01x04_Socket, J11 Conn_01x04_Socket, J12 Conn_01x06, J13 Conn_02x40_Top_Bottom, J2 USB_C_Receptacle_USB2.0_14P, J3 Conn_Coaxial_Small, J4 Conn_Coaxial_Small, J5 Conn_01x06_Socket, J6 Conn_01x02_Socket, J7 Conn_ARM_SWD_TagConnect_TC2030, J8 Conn_01x08_Socket, J9 Conn_01x04_Socket, Q1 FDMC8032L, Q2 FDMC8032L, Q3 SiR696DP, SW1 SW_SPST, U1 BQ25792RQMR, U10 INA280A1xDCK, U11 INA280A1xDCK, U12 INA280A1xDCK, U13 STM32G474VEHx, U14 APS6404L-SQRx-ZR, U15 APS6404L-SQRx-ZR, U16 AT24CS32-XHM, U17 TL3116, U2 TPS55289RYQR, U3 TPS54240DRC, U4 TPS73733DCQR, U5 OPA2325, U6 LP5907MFX-3.3, U7 OPA2356xxDGK, U8 OPA356xxDBV, U9 INA280A1xDCK, Y1 16Mhz

Commit message: Finish first schematic resivion of the SOM
Parts:
- removed J10, J11, J9: Conn_01x04_Socket, Connector_PinHeader_2.54mm:PinHeader_1x04_P2.54mm_Horizontal
- removed J12: Conn_01x06, Connector_PinHeader_2.54mm:PinHeader_1x06_P2.54mm_Horizontal
- removed J13: Conn_02x40_Top_Bottom, ul_FX18-80P-0-8SV10:CONN_FX18-80P_HIR
- removed J4: Conn_Coaxial_Small, Connector_Coaxial:SMA_Molex_73251-1153_EdgeMount_Horizontal
- removed J5: Conn_01x06_Socket, Connector_PinHeader_2.54mm:PinHeader_1x06_P2.54mm_Horizontal
- removed J6: Conn_01x02_Socket, Connector_AMASS:AMASS_XT30PW-M_1x02_P2.50mm_Horizontal
- removed J8: Conn_01x08_Socket, Connector_JST:JST_XH_B8B-XH-AM_1x08_P2.50mm_Vertical
- added C87: 100nF, Capacitor_SMD:C_0402_1005Metric, F.Cu at (177.8, 172.5)
- added C88: 100nF, Capacitor_SMD:C_0402_1005Metric, F.Cu at (177.8, 174.4)
- added C89: 100nF, Capacitor_SMD:C_0402_1005Metric, F.Cu at (177.8, 176.4)
- added D24: ESD9B3.3ST5G, Diode_SMD:D_SOD-923, F.Cu at (177.8, 183.0)
- added R60: 10K, Resistor_SMD:R_0402_1005Metric, F.Cu at (166.5, 172.5)
- added R61: 20K, Resistor_SMD:R_0402_1005Metric, F.Cu at (166.5, 174.5)
- added R62: 10K, Resistor_SMD:R_0402_1005Metric, F.Cu at (166.5, 176.5)
- added R63: 100K, Resistor_SMD:R_0402_1005Metric, F.Cu at (166.5, 178.5)
- added R64: 100K, Resistor_SMD:R_0402_1005Metric, F.Cu at (166.5, 180.4)
- added R65: 10K, Resistor_SMD:R_0402_1005Metric, F.Cu at (166.5, 182.4)
- added R66: 10K, Resistor_SMD:R_0402_1005Metric, F.Cu at (166.5, 184.4)
- added TP1: TestPoint_Probe, TestPoint:TestPoint_Pad_D2.0mm, F.Cu at (167.1, 147.2)
- added TP10: TestPoint_Probe, TestPoint:TestPoint_Pad_D2.0mm, F.Cu at (171.1, 159.4)
- added TP11: TestPoint_Probe, TestPoint:TestPoint_Pad_D2.0mm, F.Cu at (171.1, 163.4)
- added TP12: TestPoint_Probe, TestPoint:TestPoint_Pad_D2.0mm, F.Cu at (171.1, 167.5)
- added TP13: TestPoint_Probe, TestPoint:TestPoint_Pad_D2.0mm, F.Cu at (175.2, 147.2)
- added TP14: TestPoint_Probe, TestPoint:TestPoint_Pad_D2.0mm, F.Cu at (175.2, 151.3)
- added TP15: TestPoint_Probe, TestPoint:TestPoint_Pad_D2.0mm, F.Cu at (175.2, 155.3)
- added TP16: TestPoint_Probe, TestPoint:TestPoint_Pad_D2.0mm, F.Cu at (175.2, 159.4)
- added TP17: TestPoint_Probe, TestPoint:TestPoint_Pad_D2.0mm, F.Cu at (175.2, 163.4)
- added TP18: TestPoint_Probe, TestPoint:TestPoint_Pad_D2.0mm, F.Cu at (175.2, 167.5)
- added TP2: TestPoint_Probe, TestPoint:TestPoint_Pad_D2.0mm, F.Cu at (167.1, 151.3)
- added TP3: TestPoint_Probe, TestPoint:TestPoint_Pad_D2.0mm, F.Cu at (167.1, 155.3)
- added TP4: TestPoint_Probe, TestPoint:TestPoint_Pad_D2.0mm, F.Cu at (167.1, 159.4)
- added TP5: TestPoint_Probe, TestPoint:TestPoint_Pad_D2.0mm, F.Cu at (167.1, 163.4)
- added TP6: TestPoint_Probe, TestPoint:TestPoint_Pad_D2.0mm, F.Cu at (167.1, 167.5)
- added TP7: TestPoint_Probe, TestPoint:TestPoint_Pad_D2.0mm, F.Cu at (171.1, 147.2)
- added TP8: TestPoint_Probe, TestPoint:TestPoint_Pad_D2.0mm, F.Cu at (171.1, 151.3)
- added TP9: TestPoint_Probe, TestPoint:TestPoint_Pad_D2.0mm, F.Cu at (171.1, 155.3)
- added U18: OPA2356xxDGK, Package_SO:SOIC-8_3.9x4.9mm_P1.27mm, F.Cu at (172.2, 174.9)
- added U19: OPA2325, Package_SO:SOIC-8_3.9x4.9mm_P1.27mm, F.Cu at (172.2, 181.4)
- added U20: OPA356xxDBV, Package_TO_SOT_SMD:SOT-23-5, F.Cu at (179.0, 179.8)
- J3: value Conn_Coaxial_Small -> FX18-120P-0.8SV; footprint Connector_Coaxial:SMA_Molex_73251-1153_EdgeMount_Horizontal -> FX18-120P-0.8SV:HIROSE_FX18-120P-0.8SV
- moved J3 189.6 mm to (195.8, 139.8)
- moved C2 159.1 mm to (156.6, 131.3), turned to 0 degrees
- moved R2 158.4 mm to (151.5, 131.3), turned to 0 degrees
- moved J2 157.6 mm to (156.2, 140.5), turned to 0 degrees
- moved C1 156.9 mm to (147.1, 130.5), turned to 0 degrees
- moved D1 152.3 mm to (154.5, 126.7), turned to -90 degrees
- moved Q1 152.0 mm to (149.4, 127.0), turned to 180 degrees
- moved R1 150.4 mm to (156.9, 125.0), turned to 0 degrees
- moved C3 145.5 mm to (155.9, 121.7), turned to 0 degrees
- moved R3 144.8 mm to (150.9, 121.7), turned to 0 degrees
- moved SW1 143.8 mm to (162.8, 118.7), turned to 180 degrees
- moved C4 143.6 mm to (147.1, 121.1), turned to 0 degrees
- moved D2 139.3 mm to (154.6, 117.4), turned to -90 degrees
- moved Q2 139.0 mm to (149.4, 117.7), turned to 180 degrees
- moved R4 137.4 mm to (157.0, 115.8), turned to 0 degrees
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Connections:
- C4 pad 1: /Power supply/VBUS2 -> VBUS_DOCK
- C55 pad 2: /Power supply/VOUT -> VOUT
- J3 pad 1: FB_IN -> unconnected-(J3-Pad1)
- J3 pad 2: GND -> unconnected-(J3-Pad2)
- Q2 pad 5: /Power supply/VBUS2 -> VBUS_DOCK
- R17 pad 2: /Power supply/VOUT -> VOUT
- R26 pad 2: /Power supply/VOUT -> VOUT
- R3 pad 1: /Power supply/VBUS2 -> VBUS_DOCK
- U1 pad 8: /Power supply/VBUS2 -> VBUS_DOCK
- U13 pad A1: /Controller/LCD_SS -> LCD_SS
- U13 pad C2: /Controller/LCD_MOSI -> LCD_MOSI
- U13 pad C3: /Controller/LCD_SCK -> LCD_SCK
- U13 pad F1: unconnected-(U13-PC2-PadF1) -> /Analog preprocess/FB_OCD2_RECTIFIED
- U13 pad H5: /Controller/LCD_BL -> LCD_BL
- U13 pad H6: /Controller/LCD_DC -> LCD_DC
- U13 pad J1: /Controller/DAC_CH2 -> DAC_OUT
- U13 pad K6: /Controller/LCD_RST -> LCD_RST
Other:
- board outline added: 61.4 x 94 mm
