File: pcb/resoncance_converter_controller/resoncance_converter_controller.kicad_sch (KiCad schematic)
At the start: 32 parts, among them J10 Conn_01x04_Socket, J11 Conn_01x04_Socket, J12 Conn_01x06, J13 Conn_02x40_Top_Bottom, J2 USB_C_Receptacle_USB2.0_14P, J3 Conn_Coaxial_Small, J4 Conn_Coaxial_Small, J5 Conn_01x06_Socket, J6 Conn_01x02_Socket, J7 Conn_ARM_SWD_TagConnect_TC2030, J8 Conn_01x08_Socket, J9 Conn_01x04_Socket

Commit message: Finish first schematic resivion of the SOM
Parts:
- removed J10, J11, J9: Conn_01x04_Socket, Connector_PinHeader_2.54mm:PinHeader_1x04_P2.54mm_Horizontal, symbol Connector:Conn_01x04_Socket
- removed J12: Conn_01x06, Connector_PinHeader_2.54mm:PinHeader_1x06_P2.54mm_Horizontal, symbol Connector_Generic:Conn_01x06
- removed J13: Conn_02x40_Top_Bottom, ul_FX18-80P-0-8SV10:CONN_FX18-80P_HIR, symbol Connector_Generic:Conn_02x40_Top_Bottom
- removed J3, J4: Conn_Coaxial_Small, Connector_Coaxial:SMA_Molex_73251-1153_EdgeMount_Horizontal, symbol Connector:Conn_Coaxial_Small
- removed J5: Conn_01x06_Socket, Connector_PinHeader_2.54mm:PinHeader_1x06_P2.54mm_Horizontal, symbol Connector:Conn_01x06_Socket
- removed J6: Conn_01x02_Socket, Connector_AMASS:AMASS_XT30PW-M_1x02_P2.50mm_Horizontal, symbol Connector:Conn_01x02_Socket
- removed J8: Conn_01x08_Socket, Connector_PinHeader_2.54mm:PinHeader_1x08_P2.54mm_Horizontal, symbol Connector:Conn_01x08_Socket
- added D25, D26, D27, D28, D29, D30, D31, D32, D33, D34: ESD9B3.3ST5G, Diode_SMD:D_SOD-923, symbol Diode:ESD9B3.3ST5G
- added J3: FX18-120P-0.8SV, FX18-120P-0.8SV:HIROSE_FX18-120P-0.8SV, symbol FX18-120P-0.8SV:FX18-120P-0.8SV
- added R30, R70: R, Resistor_SMD:R_0402_1005Metric, symbol Device:R
- added TP1, TP10, TP11, TP12, TP13, TP14, TP15, TP16, TP17, TP18, TP2, TP3, TP4, TP5, TP6, TP7, TP8, TP9: TestPoint_Probe, TestPoint:TestPoint_Pad_D2.0mm, symbol Connector:TestPoint_Probe
Connections:
- net +BATT: now also J3.15, J3.16, J3.17, J3.18, J3.19, J3.20, J3.MFB_1, J3.MFB_2
- net CTRL_RX: now also J3.95
- net CTRL_TX: now also J3.97
- net FB_IN: now also J3.62, TP1.1
- net GND: now also D25.2 (A2), D26.2 (A2), D27.2 (A2), D28.2 (A2), D29.2 (A2), D30.2 (A2), D31.2 (A2), D32.2 (A2), D33.2 (A2), D34.2 (A2), J3.1, J3.10, J3.106, J3.107, J3.109, J3.111, J3.113, J3.115, J3.117, J3.119, J3.12, J3.120, J3.13, J3.14, J3.2, J3.21, J3.25, J3.26, J3.28, J3.29, J3.31, J3.33, J3.35, J3.37, J3.39, J3.4, J3.46, J3.47, J3.48, J3.50, J3.52, J3.54, J3.56, J3.58, J3.6, J3.60, J3.61, J3.63, J3.65, J3.67, J3.69, J3.71, J3.73, J3.74, J3.8, J3.81, J3.85, J3.86, J3.87, J3.88, J3.90, J3.92, J3.94, J3.96, J3.98
- net I2C_EXT_SCL: now also J3.93
- net I2C_EXT_SDA: now also J3.34
- net ISENSE_1: now also J3.66, TP5.1
- net ISENSE_2: now also J3.7, TP6.1
- net ISENSE_3: now also J3.68, TP7.1
- net ISENSE_4: now also J3.9, TP8.1
- net MCO: now also J3.27
- net OCD_IN: now also J3.3, TP2.1
- net OUT1: now also J3.59, TP15.1
- net OUT2: now also J3.57, TP16.1
- net OUT3: now also J3.55, TP17.1
- net OUT4: now also J3.53, TP18.1
- net OUT_SYNC_1+: now also J3.51, TP9.1
- net OUT_SYNC_1-: now also J3.110, TP10.1
- net OUT_SYNC_2+: now also J3.112, TP11.1
- net OUT_SYNC_2-: now also J3.114, TP12.1
- net OUT_SYNC_3+: now also J3.116, TP13.1
- net OUT_SYNC_3-: now also J3.118, TP14.1
- net VSENSE_IN: now also J3.64, TP4.1
- new net AUX_PWM_CH1: D33.1 (A1), J3.108, R30.2
- new net AUX_PWM_CH2: D34.1 (A1), J3.49, R70.2
- new net AUX_RX: J3.36
- new net AUX_TX: J3.38
- new net Controller/AUX_PWM_CH1: R30.1
- new net Controller/AUX_PWM_CH2: R70.1
- new net DAC_OUT: J3.72
- new net ENCODER_CHA: J3.101
- new net ENCODER_CHB: J3.41
- new net FAN_PWM: J3.100
- new net GPIO0: D29.1 (A1), J3.105
- new net GPIO1: D30.1 (A1), J3.104
- new net GPIO2: D31.1 (A1), J3.103
- new net GPIO3: D32.1 (A1), J3.102
- new net GPIO4: D25.1 (A1), J3.42
- new net GPIO5: D26.1 (A1), J3.43
- new net GPIO6: D27.1 (A1), J3.44
- new net GPIO7: D28.1 (A1), J3.45
- new net HRTIM_EEV9: J3.70
- new net HRTIM_FLT3: J3.11
- new net LCD_BL: J3.40
- new net LCD_DC: J3.30
- new net LCD_MOSI: J3.91
- new net LCD_RST: J3.99
- new net LCD_SCK: J3.32
- new net LCD_SS: J3.89
- new net OCD2_IN: J3.5, TP3.1
- new net VBUS_DOCK: J3.75, J3.76, J3.77, J3.78, J3.79, J3.80, J3.MFA_2
- new net VOUT: J3.22, J3.23, J3.24, J3.82, J3.83, J3.84, J3.MFA_1
- no-connect marks 2 -> 3
Other:
- sheet Analog preprocess ports: added FB_OCD2, FB_OCD2_RECTIFIED; removed none
- sheet Controller ports: added AUX_PWM_CH1, AUX_PWM_CH2, AUX_RX, AUX_TX, ENCODER_CHA, ENCODER_CHB, FAN_PWM, FB_OCD2, GPIO0, GPIO1, GPIO2, GPIO3, GPIO4, GPIO5, GPIO6, GPIO7, HRTIM_EEV9, HRTIM_FLT3, POWER_INT, VOUT_ENABLE; removed none
- moved on the sheet: D14, D15, D16, D17, D18, D19, D20, D21, D22, D23, J7, R50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
