File: pcb/resonance_converter_controller/resoncance_converter_controller.kicad_pcb (KiCad board)
At the start: 6 copper layers, 61.4 x 82.1 mm, 241 parts, among them J1 Micro_SD_Card_Det2, J2 USB_C_Receptacle_USB2.0_14P, J4 Conn_02x19_Odd_Even, J5 Conn_01x02, J6 FX18-120S-0.8SH, J7 Conn_ARM_SWD_TagConnect_TC2030, Q1 FDMC8032L, Q2 FDMC8032L, Q3 SiR696DP, SW1 SW_SPST, U1 BQ25792RQMR, U10 INA280A1xDCK, U11 INA280A1xDCK, U12 INA280A1xDCK, U13 STM32G474VEHx, U14 APS6404L-SQRx-ZR, U15 APS6404L-SQRx-ZR, U16 AT24CS32-XHM, U17 TL3116, U18 OPA2356xxDGK, U2 TPS55289RYQR, U20 OPA356xxDBV, U21 TPS2553DRVR, U22 USBLC6-2P6, U3 TPS54240DRC, U4 TPS73733DCQR, U5 OPA2325, U6 LP5907MFX-3.3, U7 OPA2356xxDGK, U8 OPA356xxDBV, U9 INA280A1xDCK, Y1 16Mhz

Commit message: Add reset handler buffer for dac and led
Parts:
- removed H5: MountingHole_Pad_MP, MountingHole:MountingHole_2.2mm_M2_Pad_Via
- added C88: 10uF, Capacitor_SMD:C_0402_1005Metric, B.Cu at (207.0, 144.8)
- added C94: 100nF, Capacitor_SMD:C_0402_1005Metric, B.Cu at (207.0, 143.9)
- added C95: 100nF, Capacitor_SMD:C_0402_1005Metric, F.Cu at (197.2, 150.0)
- added C96: 100nF, Capacitor_SMD:C_0402_1005Metric, F.Cu at (212.8, 121.0)
- added C97: 100nF, Capacitor_SMD:C_0402_1005Metric, F.Cu at (194.1, 139.3)
- added C98: 100nF, Capacitor_SMD:C_0402_1005Metric, F.Cu at (192.2, 139.0)
- added C99: 100nF, Capacitor_SMD:C_0402_1005Metric, F.Cu at (229.9, 145.7)
- added D35: ESD9B3.3ST5G, Diode_SMD:D_SOD-923, F.Cu at (195.1, 148.1)
- added D36: WS2812B, LED_SMD:LED_WS2812B-Mini_PLCC4_3.5x3.5mm, F.Cu at (228.7, 143.0)
- added H6: MountingHole_Pad, MountingHole:MountingHole_2.2mm_M2_Pad_Via, F.Cu at (174.2, 149.1)
- added R72: 5.1K, Resistor_SMD:R_0402_1005Metric, F.Cu at (173.1, 105.6)
- added R73: 5.1K, Resistor_SMD:R_0402_1005Metric, F.Cu at (173.1, 104.6)
- added R74: 10k, Resistor_SMD:R_0402_1005Metric, F.Cu at (214.1, 121.0)
- added R75: 10k, Resistor_SMD:R_0402_1005Metric, F.Cu at (200.5, 147.8)
- added R76: 5.1K, Resistor_SMD:R_0402_1005Metric, F.Cu at (195.1, 150.0)
- added SW2: SW_SPST, Button_Switch_SMD:SW_SPST_EVQPE1, F.Cu at (214.2, 118.0)
- added U19: TMUX154ERSW, Package_DFN_QFN:UQFN-10_1.4x1.8mm_P0.4mm, F.Cu at (197.7, 147.8)
- added U23: OPA356xxDBV, Package_TO_SOT_SMD:SOT-23-5, F.Cu at (194.6, 141.9)
- added U24: AD5246BKSZ100-RL7, AD5246BKSZ100-RL7:SOT65P210X110-6N, F.Cu at (191.5, 142.1)
- H1, H2, H3, H4: value MountingHole_Pad_MP -> MountingHole_Pad
- moved H4 54.4 mm to (228.6, 149.2)
- moved D4 6.97 mm to (220.4, 110.3)
- moved C67 4.98 mm to (194.0, 137.0), turned to 180 degrees
- moved L3 4.60 mm to (214.7, 110.5)
- moved R36 3.92 mm to (190.6, 138.5)
- moved U8 3.56 mm to (191.5, 135.4)
- moved R37 3.56 mm to (194.0, 134.8)
- moved C66 1.53 mm to (189.2, 142.2), turned to 90 degrees
- moved C77 1.45 mm to (198.7, 142.9), turned to 180 degrees
- moved C52 1.20 mm to (206.2, 116.9)
- moved C53 1.20 mm to (208.9, 116.9)
- moved C39 0.88 mm to (215.8, 115.3)
- moved C78 0.83 mm to (207.0, 142.9)
Connections:
- net I2C_INT_SCL renamed INT_I2C_SCL
- net I2C_INT_SDA renamed INT_I2C_SDA
- H1 pad 1: (no net) -> GND
- H2 pad 1: (no net) -> GND
- H3 pad 1: (no net) -> GND
- H4 pad 1: (no net) -> GND
- J6 pad SH1: (no net) -> GND
- J7 pad 3: unconnected-(J7-~{RESET}-Pad3) -> /Controller/NRST
- U13 pad F3: MCO -> MCO_NRST
- U13 pad G3: unconnected-(U13-PF2-PadG3) -> MCO_NRST_SEL
- U13 pad H2: /Analog preprocess/FB_SYNC_PADDING_V -> /Controller/DAC_CH1
- U13 pad H6: GPIO5 -> /Controller/WS2812B
- U13 pad J1: DAC_OUT -> /Analog preprocess/FB_SYNC_PADDING_V
- U13 pad K10: unconnected-(U13-PD8-PadK10) -> GPIO5
- U13 pad K2: unconnected-(U13-PC4-PadK2) -> /Controller/DAC_READ_BACK
- U13 pad K5: unconnected-(U13-VREF+-PadK5) -> Net-(U13-VREF+)
Routing:
- net /Controller/NRST: track 0.00 -> 60.5 mm, vias 0 -> 5
- net +3.3VP: track 21.5 -> 53.9 mm, vias 10 -> 11
- net INT_I2C_SCL: track 72.7 -> 104.1 mm, vias 4 -> 7
- net INT_I2C_SDA: track 71.7 -> 102.6 mm, vias 4 -> 7
- net /Controller/WS2812B: track 0.00 -> 24.1 mm, vias 0 -> 2
- net GND: track 163.5 -> 179.5 mm, vias 238 -> 239
- net /Controller/DAC_READ_BACK: track 0.00 -> 15.7 mm, vias 0 -> 2
- net MCO_NRST: track 0.00 -> 13.6 mm, vias 0 -> 2
- net MCO: track 22.8 -> 9.88 mm, vias 2 -> 1
- net MCO_NRST_SEL: track 0.00 -> 12.8 mm, vias 0 -> 2
- net VAA: track 20.7 -> 32.0 mm, vias 30 -> 22
- net /Controller/DAC_CH1: track 0.00 -> 10.8 mm
- net Net-(U23--): track 0.00 -> 6.34 mm
- net CC2: track 58.4 -> 63.8 mm, vias 2 -> 3
- net /Analog preprocess/FB_OCD_RECTIFIED: track 19.3 -> 23.7 mm
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