File: pcb/resonance_converter_controller/resoncance_converter_controller.kicad_pcb (KiCad board)
At the start: 6 copper layers, 61.4 x 79.7 mm, 272 parts, among them CN1 AXK5S40047YG, J1 Micro_SD_Card_Det2, J2 USB_C_Receptacle_USB2.0_14P, J3 DF12NB_5.0_-20DP-0.5V_51_, J4 Conn_02x19_Odd_Even, J5 Conn_01x02, J6 FX18-120S-0.8SH, J7 Conn_ARM_SWD_TagConnect_TC2030, Q1 FDMC8032L, Q2 FDMC8032L, Q3 SiR696DP, SW1 SW_SPST, SW2 SW_SPST, U1 BQ25792RQMR, U10 INA169, U11 INA169, U12 MCP4441-xxxx-ST, U13 STM32G474VEHx, U14 APS6404L-SQRx-ZR, U15 APS6404L-SQRx-ZR, U16 AT24CS32-XHM, U17 TL3116, U18 OPA2356xxDGK, U19 TMUX154ERSW, U2 TPS55289RYQR, U20 OPA356xxDBV, U21 TPS2553DRVR, U22 USBLC6-2P6, U23 OPA356xxDBV, U24 MCP4441-xxxx-ST, U25 TMUX1574RSV, U26 TMUX154ERSW, U27 INA169, U28 OPA356xxDBV, U3 TPS54240DRC, U4 TPS73733DCQR, U5 OPA2325, U6 LP5907MFX-3.3, U7 OPA2356xxDGK, U8 OPA356xxDBV, U9 INA169, Y1 16Mhz

Commit message: Update pcb
Parts:
- removed C102, C104: 100nF, Capacitor_SMD:C_0402_1005Metric
- removed J2: USB_C_Receptacle_USB2.0_14P, Connector_USB:USB_C_Receptacle_GCT_USB4105-xx-A_16P_TopMnt_Horizontal
- removed Q1, Q2: FDMC8032L, Package_SO:PowerPAK_SO-8_Dual
- removed U12: MCP4441-xxxx-ST, Package_DFN_QFN:Texas_RGP0020H_VQFN-20-1EP_4x4mm_P0.5mm_EP2.4x2.4mm_ThermalVias
- removed U25: TMUX1574RSV, Package_DFN_QFN:UQFN-16_1.8x2.6mm_P0.4mm
- removed U26: TMUX154ERSW, Package_DFN_QFN:UQFN-10_1.4x1.8mm_P0.4mm
- added C106: 100nF, Capacitor_SMD:C_0402_1005Metric, F.Cu at (105.0, 82.5)
- added J8: USB_C_Receptacle_USB2.0_16P, Connector_USB:USB_C_Receptacle_GCT_USB4105-xx-A_16P_TopMnt_Horizontal, F.Cu at (89.9, 42.8)
- added Q4: Si7938DP, Package_SO:PowerPAK_SO-8_Dual, F.Cu at (111.6, 41.0)
- added Q5: Si7938DP, Package_SO:PowerPAK_SO-8_Dual, F.Cu at (102.6, 41.0)
- added U29: MCP4441-103E_ML, Package_DFN_QFN:Texas_RGP0020H_VQFN-20-1EP_4x4mm_P0.5mm_EP2.4x2.4mm_ThermalVias, F.Cu at (103.8, 91.2)
- added U30: MCP4441-103E_ML, Package_DFN_QFN:Texas_RGP0020H_VQFN-20-1EP_4x4mm_P0.5mm_EP2.4x2.4mm_ThermalVias, F.Cu at (107.0, 85.8)
- J5: moved to B.Cu
- R7: value 6.04K -> 17.4k
- U24: value MCP4441-xxxx-ST -> TMUX154ERSW; footprint Package_DFN_QFN:Texas_RGP0020H_VQFN-20-1EP_4x4mm_P0.5mm_EP2.4x2.4mm_ThermalVias -> Package_DFN_QFN:UQFN-10_1.4x1.8mm_P0.4mm
- moved U24 25.6 mm to (132.7, 88.7), turned to 90 degrees
- moved C22 9.18 mm to (138.2, 48.7), turned to 0 degrees
- moved C21 6.48 mm to (138.2, 46.2), turned to 0 degrees
- moved J5 5.00 mm to (144.5, 45.6), turned to 90 degrees
- moved Q3 4.90 mm to (138.6, 40.8)
- moved C103 4.34 mm to (104.3, 94.3), turned to 180 degrees
- moved C101 4.23 mm to (130.7, 87.8), turned to 90 degrees
- moved U22 2.55 mm to (96.2, 49.2)
- moved R76 1.05 mm to (109.5, 83.1)
- moved R72 0.57 mm to (94.0, 50.9)
- moved R73 0.57 mm to (93.0, 50.9)
Connections:
- net /Analog preprocess/ISENSE_1_OUT renamed ISENSE_1_DPOT
- net /Analog preprocess/ISENSE_2_OUT renamed ISENSE_2_DPOT
- net /Analog preprocess/ISENSE_3_OUT renamed ISENSE_3_DPOT
- net /Analog preprocess/ISENSE_4_OUT renamed ISENSE_4_DPOT
- C21 pad 1: +BATT -> BAT
- C22 pad 1: +BATT -> BAT
- C90 pad 1: Net-(U21-IN) -> VCC
- J3 pad 11: LOCAL_LCD_DC -> LCD_DC
- J3 pad 13: LOCAL_LCD_SCK -> LCD_SCK
- J3 pad 14: LOCAL_ENCODER_CHA -> ENCODER_CHA
- J3 pad 15: LOCAL_ENCODER_CHB -> ENCODER_CHB
- J3 pad 7: LOCAL_LCD_MOSI -> LCD_MOSI
- J3 pad 9: LOCAL_LCD_SS -> LCD_SS
- J6 pad 100: GND -> VOUT
- J6 pad 101: VBUS_DOCK -> VOUT
- J6 pad 102: VBUS_DOCK -> VOUT
- J6 pad 103: VBUS_DOCK -> VOUT
- J6 pad 104: VBUS_DOCK -> VOUT
- J6 pad 105: VBUS_DOCK -> VOUT
- J6 pad 106: VBUS_DOCK -> GND
- J6 pad 19: REMOTE_ENCODER_CHB -> GND
- J6 pad 20: REMOTE_LCD_DC -> GND
- J6 pad 21: LCD_BL -> GND
- J6 pad 29: REMOTE_LCD_SCK -> GND
- J6 pad 31: LCD_MISO -> GND
- J6 pad 43: VCC -> GND
- J6 pad 45: VAA -> GND
- J6 pad 47: VAA -> GND
- J6 pad 80: REMOTE_ENCODER_CHA -> GND
- J6 pad 82: LCD_RST -> GND
- J6 pad 90: REMOTE_LCD_MOSI -> GND
- J6 pad 92: REMOTE_LCD_SS -> GND
- J6 pad MF_B1: VOUT -> VBUS_DOCK
- R37 pad 1: Net-(U24D-P3A) -> FB_OCD1_AMP_ADJ
- R66 pad 1: Net-(U20--) -> FB_OCD2_AMP_ADJ
- R76 pad 1: Net-(U24A-P0A) -> VSENSE_OUT_AMP_ADJ
- U13 pad F8: unconnected-(U13-PD14-PadF8) -> USB_DAP_DIR
- U13 pad H10: LOCAL_LCD -> USB_DAP_EN
- U13 pad H4: LOCAL_ENCODER -> unconnected-(U13-PB0-PadH4)
- U20 pad 4: Net-(U20--) -> FB_OCD2_AMP_ADJ
- U21 pad 6: Net-(U21-IN) -> VCC
- U22 pad 1: /PUSB- -> /connectors/PUSB-
- U22 pad 3: /PUSB+ -> /connectors/PUSB+
- U23 pad 1: Net-(U23--) -> AUX_DAC_IMP_IN
- U23 pad 4: Net-(U23--) -> AUX_DAC_IMP_IN
- U24 pad 1: Net-(U24D-P3A) -> SWDIO
- U24 pad 10: Net-(U23--) -> USB_DAP_EN
- U24 pad 2: GND -> SWCLK
- U24 pad 3: GND -> SBU2
- U24 pad 5: INT_I2C_SCL -> SBU1
- U24 pad 6: INT_I2C_SDA -> SWDIO
- U24 pad 7: GND -> SWCLK
- U24 pad 8: DAC_OUT -> USB_DAP_DIR
- U24 pad 9: DAC_OUT -> VCC
- U28 pad 4: Net-(U24A-P0A) -> VSENSE_OUT_AMP_ADJ
- U8 pad 4: Net-(U24D-P3A) -> FB_OCD1_AMP_ADJ
Routing:
- net SBU2: track 0.00 -> 77.0 mm, vias 0 -> 2
- net SBU1: track 0.00 -> 72.6 mm, vias 0 -> 2
- net LCD_RST: track 65.7 -> 0.00 mm, vias 3 -> 0
- net REMOTE_LCD_MOSI: track 56.9 -> 0.00 mm, vias 2 -> 0
- net REMOTE_LCD_SS: track 55.5 -> 0.00 mm, vias 2 -> 0
- net REMOTE_ENCODER_CHA: track 45.8 -> 0.00 mm, vias 5 -> 0
- net LOCAL_ENCODER_CHA: track 43.2 -> 0.00 mm, vias 4 -> 0
- net REMOTE_LCD_SCK: track 41.7 -> 0.00 mm, vias 2 -> 0
- net REMOTE_ENCODER_CHB: track 39.2 -> 0.00 mm, vias 1 -> 0
- net LOCAL_LCD_SS: track 37.6 -> 0.00 mm, vias 2 -> 0
- net LOCAL_LCD_SCK: track 36.1 -> 0.00 mm, vias 2 -> 0
- net LOCAL_LCD_MOSI: track 34.8 -> 0.00 mm, vias 2 -> 0
- net LOCAL_LCD_DC: track 34.5 -> 0.00 mm, vias 2 -> 0
- net ENCODER_CHA: track 29.0 -> 62.4 mm, vias 2 -> 4
- net LCD_BL: track 32.8 -> 0.00 mm, vias 5 -> 0
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- added copper zone on B.Cu, net VOUT
- added copper zone on In3.Cu, net VOUT
