File: pcb/resonance_converter_controller/controller.kicad_sch (KiCad schematic)
At the start: 33 parts, among them J1 Micro_SD_Card_Det2, U13 STM32G474VEHx, U14 APS6404L-SQRx-ZR, U15 APS6404L-SQRx-ZR, U16 AT24CS32-XHM, U21 TPS2553DRVR, Y1 16Mhz

Commit message: Update conector in som
Parts:
- C84, C91: footprint Capacitor_SMD:C_2220_5750Metric -> Capacitor_SMD:C_1206_3216Metric
Changed lines of the file:
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@@
 			)
 		)
-		(property "Footprint" "Capacitor_SMD:C_2220_5750Metric"
+		(property "Footprint" "Capacitor_SMD:C_1206_3216Metric"
 			(at 390.8552 259.08 0)
 			(effects
@@
 			)
 		)
-		(property "Footprint" "Capacitor_SMD:C_2220_5750Metric"
+		(property "Footprint" "Capacitor_SMD:C_1206_3216Metric"
 			(at 418.7952 259.08 0)
 			(effects

Commit message: First routing without testpoints
Parts:
- C79, C80: footprint Capacitor_SMD:C_0805_2012Metric -> Capacitor_SMD:C_0402_1005Metric
Changed lines of the file:
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@@
 			)
 		)
-		(property "Footprint" "Capacitor_SMD:C_0805_2012Metric"
+		(property "Footprint" "Capacitor_SMD:C_0402_1005Metric"
 			(at 160.9852 121.92 0)
 			(effects
@@
 			)
 		)
-		(property "Footprint" "Capacitor_SMD:C_0805_2012Metric"
+		(property "Footprint" "Capacitor_SMD:C_0402_1005Metric"
 			(at 168.6052 121.92 0)
 			(effects

Commit message: Add reset handler buffer for dac and led
Parts:
- added C88: 10uF, Capacitor_SMD:C_0402_1005Metric, symbol Device:C
- added C94, C95, C96: 100nF, Capacitor_SMD:C_0402_1005Metric, symbol Device:C
- added R74, R75: 10k, Resistor_SMD:R_0402_1005Metric, symbol Device:R
- added SW2: SW_SPST, Button_Switch_SMD:SW_SPST_EVQPE1, symbol Switch:SW_SPST
- added U19: TMUX154ERSW, Package_DFN_QFN:UQFN-10_1.4x1.8mm_P0.4mm, symbol Analog_Switch:TMUX154ERSW
Connections:
- net +3.3V: now also C95.1, R74.1, U19.9 (VCC)
- net GND: now also C88.2, C94.2, C95.2, C96.2, R75.2, SW2.1 (A), U19.4 (GND), U19.5 (B), U19.8 (~{EN})
- net GPIO5: now also U13.K10 (PD8); no longer U13.H6 (PE9)
- net MCO: now also U19.2 (A1); no longer U13.F3 (PG10)
- net MCO_NRST_SEL: now reaches U13.G3 (PF2)
- net MCO_NRST_SEL: now also R75.1, U19.10 (SEL)
- net DAC_READ_BACK: now reaches U13.K2 (PC4)
- net at U13.K5 (VREF+): now also C88.1, C94.1
- new net MCO_NRST: U13.F3 (PG10), U19.3 (A)
- new net NRST: C96.1, R74.2, SW2.2 (B), U19.1 (A0)
- new net WS2812B: U13.H6 (PE9)
- no-connect marks 1 -> 3

Commit message: Add io panel and fix controller pcb
Parts:
- added R77: 10k, Resistor_SMD:R_0402_1005Metric, symbol Device:R
Connections:
- net +3.3V: now also R77.1
- net LCD_LOCAL: now reaches U13.H10 (PD11)
- net LOCAL_ENCODER: now reaches U13.H4 (PB0)
- net KEY_INT: now reaches U13.J3 (PC5)
- net KEY_INT: now also R77.2
- net AUX_ADC_OUT: now reaches U13.K1 (PA7)
Changed lines of the file:
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@@
 	)
 	(junction
+		(at 278.13 196.85)
+		(diameter 0)
+		(color 0 0 0 0)
+	)
+	(junction
 		(at 358.14 199.39)
 		(diameter 0)
@@
 	(wire
 		(pts
+			(xy 278.13 194.31) (xy 278.13 196.85)
+		)
+		(stroke
+			(width 0)
+			(type default)
+		)
+	)
+	(wire
+		(pts
 			(xy 439.42 271.78) (xy 483.87 271.78)
 		)
@@
 	(wire
 		(pts
+			(xy 278.13 184.15) (xy 278.13 186.69)
+		)
+		(stroke
+			(width 0)
+			(type default)
+		)
+	)
+	(wire
+		(pts
 			(xy 274.32 151.13) (xy 274.32 153.67)
 		)
@@
 	(wire
 		(pts
+			(xy 285.75 196.85) (xy 278.13 196.85)
+		)
+		(stroke
+			(width 0)
+			(type default)
+		)
+	)
+	(wire
+		(pts
 			(xy 314.96 100.33) (xy 323.85 100.33)
 		)
@@
 	(wire
 		(pts
+			(xy 278.13 196.85) (xy 250.19 196.85)
+		)
+		(stroke
+			(width 0)
+			(type default)
+		)
+	)
+	(wire
+		(pts
 			(xy 368.3 213.36) (xy 372.11 213.36)
 		)
@@
 		)
 	)
+	(hierarchical_label "KEY_INT"
+		(shape input)
+		(at 285.75 196.85 0)
+		(effects
+			(font
+				(size 1.27 1.27)
+			)
+			(justify left)
+		)
+	)
 	(hierarchical_label "ISENSE1"
 		(shape input)
@@
 		)
 	)
+	(hierarchical_label "LOCAL_ENCODER"
+		(shape input)
+		(at 250.19 140.97 0)
+		(effects
+			(font
+				(size 1.27 1.27)
+			)
+			(justify left)
+		)
+	)
 	(hierarchical_label "AUX_TX"
 		(shape input)
@@
 		)
 	)
+	(hierarchical_label "LCD_LOCAL"
+		(shape input)
+		(at 209.55 194.31 180)
+		(effects
+			(font
+				(size 1.27 1.27)
+			)
+			(justify right)
+		)
+	)
 	(hierarchical_label "GPIO7"
 		(shape input)
@@
 		)
 	)
+	(hierarchical_label "AUX_ADC_OUT"
+		(shape input)
+		(at 250.19 115.57 0)
+		(effects
+			(font
+				(size 1.27 1.27)
+			)
+			(justify left)
+		)
+	)
 	(hierarchical_label "OUT_SYNC_1+"
 		(shape input)
@@
 	(symbol
 		(lib_id "power:+3.3V")
+		(at 278.13 184.15 0)
+		(unit 1)
+		(exclude_from_sim no)
+		(in_bom yes)
+		(on_board yes)
+		(dnp no)
+		(fields_autoplaced yes)
+		(property "Reference" "#PWR0236"
+			(at 278.13 187.96 0)
+			(effects
+				(font
+					(size 1.27 1.27)
+				)
+				(hide yes)
+			)
+		)
+		(property "Value" "+3.3V"
+			(at 278.13 179.07 0)
+			(effects
+				(font
+					(size 1.27 1.27)
+				)
+			)
+		)
+		(property "Footprint" ""
+			(at 278.13 184.15 0)
+			(effects
+				(font
+					(size 1.27 1.27)
+				)
+				(hide yes)
+			)
+		)
+		(property "Datasheet" ""
+			(at 278.13 184.15 0)
+			(effects
+				(font
+					(size 1.27 1.27)
+				)
+				(hide yes)
+			)
+		)
+		(property "Description" "Power symbol creates a global label with name \"+3.3V\""
+			(at 278.13 184.15 0)
+			(effects
+				(font
+					(size 1.27 1.27)
+				)
+				(hide yes)
+			)
+		)
+		(pin "1"
+		)
+		(instances
+			(project "resoncance_converter_controller"
+				(path "/834b5629-1e5f-4005-abd6-bf54830363e9/15131707-a373-4e81-a819-650b2bdd47d7"
+					(reference "#PWR0236")
+					(unit 1)
+				)
+			)
+		)
+	)
+	(symbol
+		(lib_id "power:+3.3V")
 		(at 274.32 140.97 0)
 		(unit 1)
@@
 					(unit 1)
 				)
+			)
+		)
+	)
+	(symbol
+		(lib_id "Device:R")
+		(at 278.13 190.5 0)
+		(unit 1)
+		(exclude_from_sim no)
+		(in_bom yes)
+		(on_board yes)
+		(dnp no)
+		(fields_autoplaced yes)
+		(property "Reference" "R77"
+			(at 280.67 189.2299 0)
+			(effects
+				(font
+					(size 1.27 1.27)
+				)
+				(justify left)
+			)
+		)
+		(property "Value" "10k"
+			(at 280.67 191.7699 0)
+			(effects
+				(font
+					(size 1.27 1.27)
+				)
+				(justify left)
+			)
+		)
+		(property "Footprint" "Resistor_SMD:R_0402_1005Metric"
+			(at 276.352 190.5 90)
+			(effects
+				(font
+					(size 1.27 1.27)
+				)
+				(hide yes)
+			)
+		)
+		(property "Datasheet" "~"
+			(at 278.13 190.5 0)
+			(effects
+				(font
+					(size 1.27 1.27)
+				)
+				(hide yes)
+			)
+		)
+		(property "Description" "Resistor"
+			(at 278.13 190.5 0)
+			(effects
+				(font
+					(size 1.27 1.27)
+				)
+				(hide yes)
+			)
+		)
+		(pin "1"
+		)
+		(pin "2"
+		)
+		(instances
+			(project "resoncance_converter_controller"
+				(path "/834b5629-1e5f-4005-abd6-bf54830363e9/15131707-a373-4e81-a819-650b2bdd47d7"
+					(reference "R77")
+					(unit 1)
+				)

Commit message: Add digital pots to auto adjust gain
Parts:
- added C105: 100nF, Capacitor_SMD:C_0402_1005Metric, symbol Device:C
- C72, C77: footprint Capacitor_SMD:C_1206_3216Metric -> Capacitor_SMD:C_0805_2012Metric
Connections:
- net +3.3V: now also U13.D3 (VBAT), C105.1
- net GND: now also C105.2
- no-connect marks 3 -> 2
Changed lines of the file:
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@@
 	)
 	(junction
+		(at 227.33 85.09)
+		(diameter 0)
+		(color 0 0 0 0)
+	)
+	(junction
 		(at 232.41 73.66)
 		(diameter 0)
@@
 	)
 	(junction
+		(at 153.67 73.66)
+		(diameter 0)
+		(color 0 0 0 0)
+	)
+	(junction
 		(at 147.32 242.57)
 		(diameter 0)
@@
 	)
 	(no_connect
-		(at 224.79 87.63)
-	)
-	(no_connect
 		(at 124.46 252.73)
 	)
@@
 	(wire
 		(pts
+			(xy 224.79 85.09) (xy 227.33 85.09)
+		)
+		(stroke
+			(width 0)
+			(type default)
+		)
+	)
+	(wire
+		(pts
 			(xy 203.2 73.66) (xy 215.9 73.66)
 		)
@@
 	(wire
 		(pts
-			(xy 227.33 73.66) (xy 227.33 87.63)
+			(xy 227.33 73.66) (xy 227.33 85.09)
 		)
 		(stroke
@@
 	(wire
 		(pts
-			(xy 158.75 73.66) (xy 166.37 73.66)
+			(xy 153.67 73.66) (xy 166.37 73.66)
+		)
+		(stroke
+			(width 0)
+			(type default)
+		)
+	)
+	(wire
+		(pts
+			(xy 147.32 73.66) (xy 153.67 73.66)
 		)
 		(stroke
@@
 	(wire
 		(pts
+			(xy 227.33 85.09) (xy 227.33 87.63)
+		)
+		(stroke
+			(width 0)
+			(type default)
+		)
+	)
+	(wire
+		(pts
 			(xy 358.14 196.85) (xy 358.14 199.39)
 		)
@@
 	(wire
 		(pts
+			(xy 224.79 87.63) (xy 224.79 85.09)
+		)
+		(stroke
+			(width 0)
+			(type default)
+		)
+	)
+	(wire
+		(pts
 			(xy 232.41 73.66) (xy 229.87 73.66)
 		)
@@
 	(hierarchical_label "3V3"
 		(shape input)
-		(at 158.75 73.66 180)
+		(at 147.32 73.66 180)
 		(effects
 			(font
@@
 			)
 		)
-		(property "Footprint" "Capacitor_SMD:C_1206_3216Metric"
+		(property "Footprint" "Capacitor_SMD:C_0805_2012Metric"
 			(at 264.4648 81.28 0)
 			(effects
@@
 		)
 		(instances
-			(project ""
+			(project "resoncance_converter_controller"
 				(path "/834b5629-1e5f-4005-abd6-bf54830363e9/15131707-a373-4e81-a819-650b2bdd47d7"
 					(reference "#PWR0216")
@@
 		)
 		(instances
-			(project ""
+			(project "resoncance_converter_controller"
 				(path "/834b5629-1e5f-4005-abd6-bf54830363e9/15131707-a373-4e81-a819-650b2bdd47d7"
 					(reference "#PWR0139")
@@
 		)
 		(instances
-			(project ""
+			(project "resoncance_converter_controller"
 				(path "/834b5629-1e5f-4005-abd6-bf54830363e9/15131707-a373-4e81-a819-650b2bdd47d7"
 					(reference "#PWR0163")
@@
 		)
 		(instances
-			(project ""
+			(project "resoncance_converter_controller"
 				(path "/834b5629-1e5f-4005-abd6-bf54830363e9/15131707-a373-4e81-a819-650b2bdd47d7"
 					(reference "U13")
@@
 		)
 		(instances
-			(project ""
+			(project "resoncance_converter_controller"
 				(path "/834b5629-1e5f-4005-abd6-bf54830363e9/15131707-a373-4e81-a819-650b2bdd47d7"
 					(reference "#PWR0148")
@@
 		)
 		(instances
-			(project ""
+			(project "resoncance_converter_controller"
 				(path "/834b5629-1e5f-4005-abd6-bf54830363e9/15131707-a373-4e81-a819-650b2bdd47d7"
 					(reference "#PWR0162")
@@
 		)
 		(instances
-			(project ""
+			(project "resoncance_converter_controller"
 				(path "/834b5629-1e5f-4005-abd6-bf54830363e9/15131707-a373-4e81-a819-650b2bdd47d7"
 					(reference "#PWR0137")
@@
 		)
 		(instances
-			(project ""
+			(project "resoncance_converter_controller"
 				(path "/834b5629-1e5f-4005-abd6-bf54830363e9/15131707-a373-4e81-a819-650b2bdd47d7"
 					(reference "C84")
@@
 		)
 		(instances
-			(project ""
+			(project "resoncance_converter_controller"
 				(path "/834b5629-1e5f-4005-abd6-bf54830363e9/15131707-a373-4e81-a819-650b2bdd47d7"
 					(reference "#PWR0126")
@@
 	(symbol
 		(lib_id "power:GND")
+		(at 153.67 81.28 0)
+		(unit 1)
+		(exclude_from_sim no)
+		(in_bom yes)
+		(on_board yes)
+		(dnp no)
+		(fields_autoplaced yes)
+		(property "Reference" "#PWR0268"
+			(at 153.67 87.63 0)
+			(effects
+				(font
+					(size 1.27 1.27)
+				)
+				(hide yes)
+			)
+		)
+		(property "Value" "GND"
+			(at 153.67 86.36 0)
+			(effects
+				(font
+					(size 1.27 1.27)
+				)
+			)
+		)
+		(property "Footprint" ""
+			(at 153.67 81.28 0)
+			(effects
+				(font
+					(size 1.27 1.27)
+				)
+				(hide yes)
+			)
+		)
+		(property "Datasheet" ""
+			(at 153.67 81.28 0)
+			(effects
+				(font
+					(size 1.27 1.27)
+				)
+				(hide yes)
+			)
+		)
+		(property "Description" "Power symbol creates a global label with name \"GND\" , ground"
+			(at 153.67 81.28 0)
+			(effects
+				(font
+					(size 1.27 1.27)
+				)
+				(hide yes)
+			)
+		)
+		(pin "1"
+		)
+		(instances
+			(project "resoncance_converter_controller"
+				(path "/834b5629-1e5f-4005-abd6-bf54830363e9/15131707-a373-4e81-a819-650b2bdd47d7"
+					(reference "#PWR0268")
+					(unit 1)
+				)
+			)
+		)
+	)
+	(symbol
+		(lib_id "power:GND")
 		(at 163.83 137.16 0)
 		(unit 1)
@@
 		)
 		(instances
-			(project ""
+			(project "resoncance_converter_controller"
 				(path "/834b5629-1e5f-4005-abd6-bf54830363e9/15131707-a373-4e81-a819-650b2bdd47d7"
 					(reference "#PWR0125")
@@
 	)
 	(symbol
+		(lib_id "Device:C")
+		(at 153.67 77.47 0)
+		(unit 1)
+		(exclude_from_sim no)
+		(in_bom yes)
+		(on_board yes)
+		(dnp no)
+		(property "Reference" "C105"
+			(at 157.734 76.2 0)
+			(effects
+				(font
+					(size 1.27 1.27)
+				)
+				(justify left)
+			)
+		)
+		(property "Value" "100nF"
+			(at 157.734 78.74 0)
+			(effects
+				(font
+					(size 1.27 1.27)
+				)
+				(justify left)
+			)
+		)
+		(property "Footprint" "Capacitor_SMD:C_0402_1005Metric"
+			(at 154.6352 81.28 0)
+			(effects
+				(font
+					(size 1.27 1.27)
+				)
+				(hide yes)
+			)
+		)
+		(property "Datasheet" "~"
+			(at 153.67 77.47 0)
+			(effects
+				(font
+					(size 1.27 1.27)
+				)
+				(hide yes)
+			)
+		)
+		(property "Description" "Unpolarized capacitor"
+			(at 153.67 77.47 0)
+			(effects
+				(font
+					(size 1.27 1.27)
+				)
+				(hide yes)
+			)
+		)
+		(pin "2"
+		)
+		(pin "1"
+		)
+		(instances
+			(project "resoncance_converter_controller"
+				(path "/834b5629-1e5f-4005-abd6-bf54830363e9/15131707-a373-4e81-a819-650b2bdd47d7"
+					(reference "C105")
+					(unit 1)
+				)
+			)
+		)
+	)
+	(symbol
 		(lib_id "power:GND")
 		(at 323.85 262.89 0)
@@
 		)
 		(instances
-			(project ""
+			(project "resoncance_converter_controller"
 				(path "/834b5629-1e5f-4005-abd6-bf54830363e9/15131707-a373-4e81-a819-650b2bdd47d7"
 					(reference "#PWR0203")
@@
 		)
 		(instances
-			(project ""
+			(project "resoncance_converter_controller"
 				(path "/834b5629-1e5f-4005-abd6-bf54830363e9/15131707-a373-4e81-a819-650b2bdd47d7"
 					(reference "#PWR0154")
@@
 		)
 		(instances
-			(project ""
+			(project "resoncance_converter_controller"
 				(path "/834b5629-1e5f-4005-abd6-bf54830363e9/15131707-a373-4e81-a819-650b2bdd47d7"
 					(reference "#PWR0129")
@@
 		)
 		(instances
-			(project ""
+			(project "resoncance_converter_controller"
 				(path "/834b5629-1e5f-4005-abd6-bf54830363e9/15131707-a373-4e81-a819-650b2bdd47d7"
 					(reference "#PWR0138")
@@
 		)
 		(instances
-			(project ""
+			(project "resoncance_converter_controller"
 				(path "/834b5629-1e5f-4005-abd6-bf54830363e9/15131707-a373-4e81-a819-650b2bdd47d7"
 					(reference "#PWR0127")
@@
 		)
 		(instances
-			(project ""
+			(project "resoncance_converter_controller"
 				(path "/834b5629-1e5f-4005-abd6-bf54830363e9/15131707-a373-4e81-a819-650b2bdd47d7"
 					(reference "U14")
@@
 			)
 		)
-		(property "Footprint" "Capacitor_SMD:C_1206_3216Metric"
+		(property "Footprint" "Capacitor_SMD:C_0805_2012Metric"
 			(at 167.3352 81.28 0)
 			(effects
@@
 		)
 		(instances
-			(project ""
+			(project "resoncance_converter_controller"
 				(path "/834b5629-1e5f-4005-abd6-bf54830363e9/15131707-a373-4e81-a819-650b2bdd47d7"
 					(reference "#PWR0221")
@@
 		)
 		(instances
-			(project ""
+			(project "resoncance_converter_controller"
 				(path "/834b5629-1e5f-4005-abd6-bf54830363e9/15131707-a373-4e81-a819-650b2bdd47d7"
 					(reference "#PWR0160")
@@
 		)
 		(instances
-			(project ""
+			(project "resoncance_converter_controller"
 				(path "/834b5629-1e5f-4005-abd6-bf54830363e9/15131707-a373-4e81-a819-650b2bdd47d7"
 					(reference "U16")
@@
 		)
 		(instances
-			(project ""
+			(project "resoncance_converter_controller"
 				(path "/834b5629-1e5f-4005-abd6-bf54830363e9/15131707-a373-4e81-a819-650b2bdd47d7"
 					(reference "U19")
@@
 		)
 		(instances
-			(project ""
+			(project "resoncance_converter_controller"
 				(path "/834b5629-1e5f-4005-abd6-bf54830363e9/15131707-a373-4e81-a819-650b2bdd47d7"
 					(reference "#PWR0153")
@@
 		)
 		(instances
-			(project ""
+			(project "resoncance_converter_controller"
 				(path "/834b5629-1e5f-4005-abd6-bf54830363e9/15131707-a373-4e81-a819-650b2bdd47d7"
 					(reference "#PWR0224")
@@
 		)
 		(instances
-			(project ""
+			(project "resoncance_converter_controller"
 				(path "/834b5629-1e5f-4005-abd6-bf54830363e9/15131707-a373-4e81-a819-650b2bdd47d7"
 					(reference "#PWR0128")
@@
 		)
 		(instances
-			(project ""
+			(project "resoncance_converter_controller"
 				(path "/834b5629-1e5f-4005-abd6-bf54830363e9/15131707-a373-4e81-a819-650b2bdd47d7"
 					(reference "#PWR0222")
@@
 		)
 		(instances
-			(project ""
+			(project "resoncance_converter_controller"
 				(path "/834b5629-1e5f-4005-abd6-bf54830363e9/15131707-a373-4e81-a819-650b2bdd47d7"
 					(reference "#PWR0133")
