File: pcb/resonance_converter_controller/controller.kicad_sch (KiCad schematic)
At the start: 43 parts, among them J1 Micro_SD_Card_Det2, SW2 SW_SPST, U13 STM32G474VEHx, U14 APS6404L-SQRx-ZR, U15 APS6404L-SQRx-ZR, U16 AT24CS32-XHM, U19 TMUX154ERSW, U21 TPS2553DRVR, Y1 16Mhz

Commit message: Update pcb
Parts:
- added C101: 100nF, Capacitor_SMD:C_0402_1005Metric, symbol Device:C
- added U24: TMUX154ERSW, Package_DFN_QFN:UQFN-10_1.4x1.8mm_P0.4mm, symbol Analog_Switch:TMUX154ERSW
Connections:
- net +3.3V: now also C90.1, U21.6 (IN), C101.1, U24.9 (VCC)
- net GND: now also C101.2, U24.4 (GND)
- net SWCLK: now also U24.2 (A1), U24.7 (B0)
- net SWDIO: now also U24.1 (A0), U24.6 (B1)
- net USB_DAP_DIR: now reaches U13.F8 (PD14)
- net USB_DAP_DIR: now also U24.8 (~{EN})
- net LCD_LOCAL renamed USB_DAP_EN
- net USB_DAP_EN: now also U24.10 (SEL)
- net LOCAL_ENCODER: no longer names the net of U13.H4 (PB0)
- new net SBU1: U24.5 (B)
- new net SBU2: U24.3 (A)
