File: pcb/resonance_converter_controller/analog.kicad_sch (KiCad schematic)
At the start: 67 parts, among them U10 INA169, U11 INA169, U12 MCP4441-xxxx-ST, U17 TL3116, U18 OPA2356xxDGK, U20 OPA356xxDBV, U23 OPA356xxDBV, U24 MCP4441-xxxx-ST, U27 INA169, U28 OPA356xxDBV, U5 OPA2325, U7 OPA2356xxDGK, U8 OPA356xxDBV, U9 INA169

Commit message: Update pcb
Parts:
- removed C104: 100nF, Capacitor_SMD:C_0402_1005Metric, symbol Device:C
- removed U12, U24: MCP4441-xxxx-ST, Package_DFN_QFN:Texas_RGP0020H_VQFN-20-1EP_4x4mm_P0.5mm_EP2.4x2.4mm_ThermalVias, symbol Potentiometer_Digital:MCP4441-xxxx-ST
- added C106: 100nF, Capacitor_SMD:C_0402_1005Metric, symbol Device:C
- added U29, U30: MCP4441-103E_ML, Package_DFN_QFN:Texas_RGP0020H_VQFN-20-1EP_4x4mm_P0.5mm_EP2.4x2.4mm_ThermalVias, symbol JLCImport:MCP4441-103E_ML
Connections:
- net GND: now also C106.2, U29.1 (P3B), U29.10 (P0W), U29.11 (P0B), U29.16 (P2B), U29.17 (P2W), U29.20 (P3W), U29.21 (EP), U29.5 (VSS), U29.6 (P1B), U29.7 (P1W), U30.1 (P3B), U30.10 (P0W), U30.11 (P0B), U30.16 (P2B), U30.17 (P2W), U30.2 (HVC/A0), U30.20 (P3W), U30.21 (EP), U30.5 (VSS)
- net SCL: now also U29.3 (SCL), U30.3 (SCL)
- net SDA: now also U29.4 (SDA), U30.4 (SDA)
- net VCC: now also C106.1, U29.12 (WP#), U29.13 (RESET#), U29.14 (A1), U29.15 (VDD), U29.2 (HVC/A0), U30.12 (WP#), U30.13 (RESET#), U30.14 (A1), U30.15 (VDD)
- net VSENSE_OUT_AMP_ADJ: now reaches R76.1, U28.4 (-)
- net VSENSE_OUT_AMP_ADJ: now also U30.9 (P0A)
- net AUX_DAC_IMP_IN: now reaches U23.1, U23.4 (-)
- net AUX_DAC_IMP_IN: now also U30.7 (P1W), U30.8 (P1A)
- net FB_OCD1_AMP_ADJ: now reaches R37.1, U8.4 (-)
- net FB_OCD1_AMP_ADJ: now also U30.19 (P3A)
- net FB_OCD2_AMP_ADJ: now reaches R66.1, U20.4 (-)
- net FB_OCD2_AMP_ADJ: now also U30.18 (P2A)
- net DAC_OUT renamed AUX_DAC_IMP_OUT
- net AUX_DAC_IMP_OUT: now also U30.6 (P1B)
- net ISENSE_1_OUT renamed ISENSE_1_DPOT
- net ISENSE_1_DPOT: now also U29.8 (P1A)
- net ISENSE_2_OUT renamed ISENSE_2_DPOT
- net ISENSE_2_DPOT: now also U29.9 (P0A)
- net ISENSE_3_OUT renamed ISENSE_3_DPOT
- net ISENSE_3_DPOT: now also U29.18 (P2A)
- net ISENSE_4_OUT renamed ISENSE_4_DPOT
- net ISENSE_4_DPOT: now also U29.19 (P3A)
Other:
- moved on the sheet: C103, C68, C69, C70, C71, D10, D11, D12, D35, D37, D7, R78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
