File: pcb/resonance_converter_controller/power.kicad_sch (KiCad schematic)
At the start: 109 parts, among them Q1 FDMC8032L, Q2 FDMC8032L, Q3 SiR696DP, SW1 SW_SPST, U1 BQ25792RQMR, U2 TPS55289RYQR, U3 TPS54240DRC, U4 TPS73733DCQR, U6 LP5907MFX-3.3

Commit message: Update pcb
Parts:
- removed Q1, Q2: FDMC8032L, Package_SO:PowerPAK_SO-8_Dual, symbol Transistor_FET:FDMC8032L
- added Q4, Q5: Si7938DP, Package_SO:PowerPAK_SO-8_Dual, symbol Si7938DP:Si7938DP
- R7: value 6.04K -> 17.4k
Connections:
- net BAT: now also C21.1, C22.1
- net VBAT: no longer C21.1, C22.1
- net VBUS: now also Q4.6 (D2), Q5.6 (D2)
- net VBUS1: now also Q5.5 (D1)
- net VBUS2: now also Q4.5 (D1)
- net at D2.1 (K), R4.1: now also Q4.2 (G1), Q4.4 (G2)
- net at D2.2 (A): now also Q4.1 (S1), Q4.3 (S2)
- net at D1.1 (K), R1.1: now also Q5.2 (G1), Q5.4 (G2)
- net at D1.2 (A): now also Q5.1 (S1), Q5.3 (S2)
Other:
- moved on the sheet: C21, C22
