File: pcb/resonance_converter_controller/resoncance_converter_controller.kicad_sch (KiCad schematic)
At the start: 53 parts, among them CN1 AXK5S40047YG, J2 USB_C_Receptacle_USB2.0_14P, J3 DF12NB_5.0_-20DP-0.5V_51_, J4 Conn_02x19_Odd_Even, J5 Conn_01x02, J6 FX18-120S-0.8SH, J7 Conn_ARM_SWD_TagConnect_TC2030, U22 USBLC6-2P6, U25 TMUX1574RSV, U26 TMUX154ERSW

Commit message: Update pcb
Parts:
- removed C101, C102: 100nF, Capacitor_SMD:C_0402_1005Metric, symbol Device:C
- removed CN1: AXK5S40047YG, AXK5S40047YG:CONN-SMD_40P-P0.50_AXK5S40047YG, symbol AXK5S40047YG:AXK5S40047YG
- removed J2: USB_C_Receptacle_USB2.0_14P, Connector_USB:USB_C_Receptacle_GCT_USB4105-xx-A_16P_TopMnt_Horizontal, symbol Connector:USB_C_Receptacle_USB2.0_14P
- removed J3: DF12NB_5.0_-20DP-0.5V_51_, DF12NB_5.0_-20DP-0.5V_51_:HRS_DF12NB_5.0_-20DP-0.5V_51_, symbol DF12NB_5.0_-20DP-0.5V_51_:DF12NB_5.0_-20DP-0.5V_51_
- removed J4: Conn_02x19_Odd_Even, Connector_PinSocket_2.54mm:PinSocket_2x19_P2.54mm_Vertical_SMD, symbol Connector_Generic:Conn_02x19_Odd_Even
- removed J5: Conn_01x02, Connector_AMASS:AMASS_XT30U-M_1x02_P5.0mm_Vertical, symbol Connector_Generic:Conn_01x02
- removed J6: FX18-120S-0.8SH, FX18-120S-0.8SH:HIROSE_FX18-120S-0.8SH, symbol FX18-120S-0.8SH:FX18-120S-0.8SH
- removed R72, R73: 5.1K, Resistor_SMD:R_0402_1005Metric, symbol Device:R
- removed U22: USBLC6-2P6, Package_TO_SOT_SMD:SOT-666, symbol Power_Protection:USBLC6-2P6
- removed U25: TMUX1574RSV, Package_DFN_QFN:UQFN-16_1.8x2.6mm_P0.4mm, symbol Analog_Switch:TMUX1574RSV
- removed U26: TMUX154ERSW, Package_DFN_QFN:UQFN-10_1.4x1.8mm_P0.4mm, symbol Analog_Switch:TMUX154ERSW
Connections:
- net NRST renamed Controller/NRST
- net SWCLK renamed Controller/SWCLK
- net SWDIO renamed Controller/SWDIO
Other:
- added sheet connectors (connectors.kicad_sch)
- sheet Controller ports: added none; removed LCD_LOCAL, LOCAL_ENCODER
- moved on the sheet: C99, D14, D15, D16, D17, D18, D19, D20, D21, D22, D23, D25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
