File: pcb/resonance_converter_controller_debug_probe/connectors.kicad_sch (KiCad schematic)
At the start: 2 parts, among them J6 FX18-120S-0.8SH, J8 Conn_01x15

Commit message: Add schematic for debug probe
Parts:
- J8: footprint (none) -> Connector_FFC-FPC:Hirose_FH12-15S-0.5SH_1x15-1MP_P0.50mm_Horizontal
Changed lines of the file:
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@@
 			)
 		)
-		(property "Footprint" ""
+		(property "Footprint" "Connector_FFC-FPC:Hirose_FH12-15S-0.5SH_1x15-1MP_P0.50mm_Horizontal"
 			(at 257.81 69.85 0)
 			(effects
