File: pcb/resonance_converter_controller_debug_probe/eth.kicad_sch (KiCad schematic)
At the start: 52 parts, among them J2 SFP, J7 RJ45_JK00177, U24 DP83869HM, U25 LP5912-1.1DRV, U26 LP5912-1.8DRV, U29 LP5912-2.5DRV, Y1 Crystal_GND24

Commit message: Add schematic for debug probe
Parts:
- C88: footprint (none) -> Capacitor_SMD:CP_Elec_6.3x3
- J2: footprint (none) -> Connector:Connector_SFP_and_Cage
Changed lines of the file:
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@@
 			)
 		)
-		(property "Footprint" ""
+		(property "Footprint" "Connector:Connector_SFP_and_Cage"
 			(at 248.92 77.47 0)
 			(effects
@@
 			)
 		)
-		(property "Footprint" ""
+		(property "Footprint" "Capacitor_SMD:CP_Elec_6.3x3"
 			(at 30.1752 119.38 0)
 			(effects

Commit message: Fix schematic and initial component layout
Parts:
- added C149, C151, C153, C155: 100nF, Capacitor_SMD:C_0402_1005Metric, symbol Device:C
- added C150, C152, C154, C156: 1u, Capacitor_SMD:C_0402_1005Metric, symbol Device:C
- C67, C73, C76, C77, C79: footprint Capacitor_SMD:C_0805_2012Metric -> Capacitor_SMD:C_0402_1005Metric
- C88: footprint Capacitor_SMD:CP_Elec_6.3x3 -> Capacitor_SMD:C_1206_3216Metric
Connections:
- net +1V1: now also C153.1, C154.1, C155.1, C156.1
- net +2V5: now also C149.1, C150.1
- net +3.3V: now also C151.1, C152.1
- net GND: now also C149.2, C150.2, C151.2, C152.2, C153.2, C154.2, C155.2, C156.2
Other:
- moved on the sheet: C74, C75, C76, C77, C82, C83
