File: pcb/resonance_converter_controller_debug_probe/memory.kicad_sch (KiCad schematic)
At the start: 11 parts, among them J10 Micro_SD_Card_Det2, J9 Micro_SD_Card_Det2, U31 TPS2553DRVR

Commit message: Fix schematic and initial component layout
Connections:
- net +3.3V: now also C105.1, U31.6 (IN)
