File: pcb/resonance_converter_controller_debug_probe/power.kicad_sch (KiCad schematic)
At the start: 62 parts, among them Q4 Q_NMOS_GDS, U1 TPS2121RUXR, U23 TPS2412D, U3 TPS56637RPAR, U4 TPS73733DCQR, U5 TPS259474ARPWR, U6 LP5907MFX-3.3

Commit message: Add schematic for debug probe
Parts:
- U23: footprint (none) -> Package_SO:TSSOP-8_4.4x3mm_P0.65mm
Changed lines of the file:
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@@
 			)
 		)
-		(property "Footprint" ""
+		(property "Footprint" "Package_SO:TSSOP-8_4.4x3mm_P0.65mm"
 			(at 306.07 50.8 0)
 			(effects

Commit message: Fix schematic and initial component layout
Parts:
- added C157, C158, C159: C_Polarized, Capacitor_SMD:C_2220_5750Metric, symbol Device:C_Polarized
- C2, C3: footprint Capacitor_SMD:CP_Elec_10x10 -> Capacitor_SMD:C_2220_5750Metric
Connections:
- net +5V: now also C159.1
- net GND: now also C157.2, C158.2, C159.2
- net VPP: now also C157.1, C158.1
