File: pcb/resonance_converter_controller_dock_v1/resonance_converter_controller_dock_v1.kicad_pcb (KiCad board)
At the start: 4 copper layers, 161.3 x 151.8 mm, 167 parts, among them J1 Conn_01x04, J10 Conn_Coaxial, J11 Conn_01x02, J12 Conn_01x02, J13 Conn_Coaxial, J14 Conn_Coaxial, J15 Conn_01x02, J16 Conn_01x02, J17 Conn_Coaxial, J18 Conn_01x02, J19 Conn_01x04, J2 Conn_01x52_MountingPin, J20 Conn_01x04, J21 Conn_01x04, J22 Conn_01x06, J23 Conn_Coaxial, J24 Conn_01x02, J25 Conn_01x02, J26 Conn_Coaxial, J27 Conn_01x04, J28 Conn_01x02, J29 USB_C_Receptacle_USB2.0_14P, J3 Conn_Coaxial, J30 Conn_01x09, J31 Conn_01x04, J32 Conn_01x04, J34 Conn_02x05_Odd_Even, J35 FX18-120P-0.8SV, J4 Conn_01x02, J5 Conn_Coaxial, J6 Conn_01x02, J7 Conn_Coaxial, J8 Conn_01x02, J9 Conn_Coaxial, M1 Fan_4pin, SW1 RotaryEncoder_Switch_MP, SW2 SW_SPST, SW3 SW_SPST, SW4 SW_SPST, SW5 SW_SPST, SW6 SW_SPST, U1 STM32F105R8Tx, U10 TMUX131RMG, U11 TMUX131RMG, U12 TMUX131RMG, U13 TMUX131RMG, U14 TMUX131RMG, U15 TMUX154ERSW, U16 AT24CS32-XHM, U17 TMUX1574RSV, U18 TMUX1574RSV, U19 TMUX131RMG, U2 FUSB302B01MPX, U20 TMUX1574RSV, U21 TMUX154ERSW, U22 TMUX154ERSW, U23 TMUX154ERSW, U24 BTS5012SDA, U25 BTS5012SDA, U26 BTS5012SDA, U27 74LVC1G04, U3 LM2576HVS-ADJ, U4 TMUX131RMG, U5 LM7812_TO220, U6 TPS2116DRL, U7 AZ1117-3.3, U8 AP2171W, U9 TMUX131RMG, Y1 16Mhz

Commit message: Update pcb
Parts:
- added J33: Conn_02x09_Top_Bottom, Connector_PinHeader_2.54mm:PinHeader_2x09_P2.54mm_Vertical, F.Cu at (214.2, 151.2)
- added J36: Conn_02x09_Top_Bottom, Connector_PinHeader_2.54mm:PinHeader_2x09_P2.54mm_Vertical, F.Cu at (217.1, 112.6)
- added J37: Conn_01x04, Connector_PinHeader_2.54mm:PinHeader_1x04_P2.54mm_Vertical, F.Cu at (219.4, 106.7)
- added J38: Conn_01x04, Connector_PinHeader_2.54mm:PinHeader_1x04_P2.54mm_Vertical, F.Cu at (161.5, 123.5)
- added R23: 5.1K, Resistor_SMD:R_0402_1005Metric, F.Cu at (222.3, 25.3)
- added R24: 5.1K, Resistor_SMD:R_0402_1005Metric, F.Cu at (222.3, 30.9)
- added R28: 10K, Resistor_SMD:R_0402_1005Metric, F.Cu at (183.7, 67.7)
- added SW7: SW_SPST, Button_Switch_SMD:SW_SPST_EVQPE1, F.Cu at (183.8, 72.3)
Connections:
- U1 pad 60: unconnected-(U1-BOOT0-Pad60) -> Net-(SW7-A)
Routing:
- net INTERNAL_I2C_SCL: track 139.4 -> 7.48 mm, vias 2 -> 0
- net INTERNAL_I2C_SDA: track 140.3 -> 10.3 mm, vias 3 -> 0
- net INTR: track 93.7 -> 0.00 mm, vias 2 -> 0
- net SYNC: track 92.9 -> 0.00 mm, vias 2 -> 0
- net /LOCK: track 92.3 -> 0.00 mm, vias 2 -> 0
- net GND: track 195.3 -> 267.1 mm, vias 164 -> 165
- net VBUS_DOCK: track 284.1 -> 306.5 mm, vias 5 -> 14
- net +3.3V: track 46.6 -> 64.0 mm
- net Net-(SW7-A): track 0.00 -> 14.4 mm
- net VOUT: track 224.2 -> 233.8 mm, vias 2 -> 5
- net DEV_PAD_CENTER: track 190.1 -> 181.7 mm
- net DEV_ENCODER_B: track 175.3 -> 169.2 mm
- net DEV_ENCODER_A: track 173.2 -> 167.3 mm
- net OUT1: track 64.5 -> 67.8 mm
- net Net-(J29-CC1): track 9.84 -> 12.6 mm
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Other:
- board size 161.3 x 151.8 mm -> 166.4 x 156.2 mm
