File: pcb/resonance_converter_controller_dock_v1/resonance_converter_controller_dock_v1.kicad_sch (KiCad schematic)
At the start: 167 parts, among them J1 Conn_01x04, J10 Conn_Coaxial, J11 Conn_01x02, J12 Conn_01x02, J13 Conn_Coaxial, J14 Conn_Coaxial, J15 Conn_01x02, J16 Conn_01x02, J17 Conn_Coaxial, J18 Conn_01x02, J19 Conn_01x04, J2 Conn_01x52_MountingPin, J20 Conn_01x04, J21 Conn_01x04, J22 Conn_01x06, J23 Conn_Coaxial, J24 Conn_01x02, J25 Conn_01x02, J26 Conn_Coaxial, J27 Conn_01x04, J28 Conn_01x02, J29 USB_C_Receptacle_USB2.0_14P, J3 Conn_Coaxial, J30 Conn_01x09, J31 Conn_01x04, J32 Conn_01x04, J34 Conn_02x05_Odd_Even, J35 FX18-120P-0.8SV, J4 Conn_01x02, J5 Conn_Coaxial, J6 Conn_01x02, J7 Conn_Coaxial, J8 Conn_01x02, J9 Conn_Coaxial, M1 Fan_4pin, SW1 RotaryEncoder_Switch_MP, SW2 SW_SPST, SW3 SW_SPST, SW4 SW_SPST, SW5 SW_SPST, SW6 SW_SPST, U1 STM32F105R8Tx, U10 TMUX131RMG, U11 TMUX131RMG, U12 TMUX131RMG, U13 TMUX131RMG, U14 TMUX131RMG, U15 TMUX154ERSW, U16 AT24CS32-XHM, U17 TMUX1574RSV, U18 TMUX1574RSV, U19 TMUX131RMG, U2 FUSB302B01MPX, U20 TMUX1574RSV, U21 TMUX154ERSW, U22 TMUX154ERSW, U23 TMUX154ERSW, U24 BTS5012SDA, U25 BTS5012SDA, U26 BTS5012SDA, U27 74LVC1G04, U3 LM2576HVS-ADJ, U4 TMUX131RMG, U5 LM7812_TO220, U6 TPS2116DRL, U7 AZ1117-3.3, U8 AP2171W, U9 TMUX131RMG, Y1 16Mhz

Commit message: Update pcb
Parts:
- added J33, J36: Conn_02x09_Top_Bottom, Connector_PinHeader_2.54mm:PinHeader_2x09_P2.54mm_Vertical, symbol Connector_Generic:Conn_02x09_Top_Bottom
- added J37, J38: Conn_01x04, Connector_PinHeader_2.54mm:PinHeader_1x04_P2.54mm_Vertical, symbol Connector_Generic:Conn_01x04
- added R23, R24: 5.1K, Resistor_SMD:R_0402_1005Metric, symbol Device:R
- added R28: 10K, Resistor_SMD:R_0402_1005Metric, symbol Device:R
- added SW7: SW_SPST, Button_Switch_SMD:SW_SPST_EVQPE1, symbol Switch:SW_SPST
Connections:
- net +3.3V: now also J33.1 (Pin_1), J36.1 (Pin_1), J37.1 (Pin_1), J38.1 (Pin_1), SW7.2 (B)
- net FROM_REMOTE_CTRL_RX: now also J36.16 (Pin_16)
- net FROM_REMOTE_CTRL_TX: now also J33.17 (Pin_17)
- net FROM_REMOTE_ENCODER_A: now also J36.9 (Pin_9)
- net FROM_REMOTE_ENCODER_B: now also J36.10 (Pin_10)
- net FROM_REMOTE_LCD_BL: now also J33.2 (Pin_2)
- net FROM_REMOTE_LCD_DC: now also J33.7 (Pin_7)
- net FROM_REMOTE_LCD_MISO: now also J36.3 (Pin_3)
- net FROM_REMOTE_LCD_MOSI: now also J33.5 (Pin_5)
- net FROM_REMOTE_LCD_RST: now also J33.8 (Pin_8)
- net FROM_REMOTE_LCD_SCK: now also J33.4 (Pin_4)
- net FROM_REMOTE_LCD_SS: now also J33.6 (Pin_6)
- net FROM_REMOTE_PAD_CENTER: now also J36.15 (Pin_15)
- net FROM_REMOTE_PAD_DOWN: now also J36.12 (Pin_12)
- net FROM_REMOTE_PAD_LEFT: now also J36.13 (Pin_13)
- net FROM_REMOTE_PAD_RIGHT: now also J36.14 (Pin_14)
- net FROM_REMOTE_PAD_UP: now also J36.11 (Pin_11)
- net GND: now also J33.18 (Pin_18), J36.18 (Pin_18), J37.4 (Pin_4), J38.4 (Pin_4), R23.2, R24.2, R28.2
- net I2C_EXT_SCL: now also J38.3 (Pin_3)
- net I2C_EXT_SDA: now also J38.2 (Pin_2)
- net INTERNAL_I2C_SCL: now also J37.3 (Pin_3)
- net INTERNAL_I2C_SDA: now also J37.2 (Pin_2)
- net TO_REMOTE_CTRL_RX: now also J33.16 (Pin_16)
- net TO_REMOTE_CTRL_TX: now also J36.17 (Pin_17)
- net TO_REMOTE_ENCODER_A: now also J33.9 (Pin_9)
- net TO_REMOTE_ENCODER_B: now also J33.10 (Pin_10)
- net TO_REMOTE_LCD_BL: now also J36.2 (Pin_2)
- net TO_REMOTE_LCD_DC: now also J36.7 (Pin_7)
- net TO_REMOTE_LCD_MISO: now also J33.3 (Pin_3)
- net TO_REMOTE_LCD_MOSI: now also J36.5 (Pin_5)
- net TO_REMOTE_LCD_RST: now also J36.8 (Pin_8)
- net TO_REMOTE_LCD_SCK: now also J36.4 (Pin_4)
- net TO_REMOTE_LCD_SS: now also J36.6 (Pin_6)
- net TO_REMOTE_PAD_CENTER: now also J33.15 (Pin_15)
- net TO_REMOTE_PAD_DOWN: now also J33.12 (Pin_12)
- net TO_REMOTE_PAD_LEFT: now also J33.13 (Pin_13)
- net TO_REMOTE_PAD_RIGHT: now also J33.14 (Pin_14)
- net TO_REMOTE_PAD_UP: now also J33.11 (Pin_11)
- net at C31.1, J29.A5 (CC1), U2.10 (CC1)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: now also R23.1
- net at C32.1, J29.B5 (CC2), U2.1 (CC2)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: now also R24.1
- net at U1.60 (BOOT0): now also R28.1, SW7.1 (A)
Other:
- moved on the sheet: C36, U2
