File: pcb/resonance_converter_controller_io/resonance_converter_controller_io.kicad_pcb (KiCad board)
At the start: 4 copper layers, 61.4 x 79.6 mm, 53 parts, among them J1 DF12NB_5.0_-20DP-0.5V_51_, J2 Conn_01x30_MountingPin, J3 Conn_01x02, J4 Conn_01x02, J7 Conn_ARM_SWD_TagConnect_TC2030, SW1 RotaryEncoder_Switch_MP, SW2 SW_SPST, SW3 SW_SPST, SW4 SW_SPST, SW5 SW_SPST, U1 PCF8574RGTR, U2 TLV61047DDC, U3 AXK6S40647YG

Commit message: Update pcb
Parts:
- added C19: 100nF, Capacitor_SMD:C_0402_1005Metric, F.Cu at (147.5, 64.3)
- added C20: 100nF, Capacitor_SMD:C_0402_1005Metric, F.Cu at (109.3, 65.3)
- moved J4 10.1 mm to (154.1, 94.7)
- moved J3 10.0 mm to (154.1, 104.8)
Connections:
- U3 pad 21: VSYS -> VOUT
- U3 pad 22: VOUT -> VSYS
- U3 pad 23: VSYS -> VOUT
- U3 pad 24: VOUT -> VSYS
- U3 pad 25: VSYS -> VOUT
- U3 pad 26: VOUT -> VSYS
- U3 pad 27: VSYS -> VOUT
- U3 pad 28: VOUT -> VSYS
- U3 pad 29: VSYS -> VOUT
- U3 pad 30: VOUT -> VSYS
- U3 pad 31: VSYS -> VOUT
- U3 pad 32: VOUT -> VSYS
- U3 pad 33: VSYS -> VOUT
- U3 pad 34: VOUT -> VSYS
- U3 pad 35: VSYS -> VOUT
- U3 pad 36: VOUT -> VSYS
- U3 pad 37: VSYS -> VOUT
- U3 pad 38: VOUT -> VSYS
- U3 pad 39: VSYS -> VOUT
- U3 pad 40: VOUT -> VSYS
Routing:
- net VSYS: track 73.0 -> 65.1 mm
- net VOUT: track 65.1 -> 73.0 mm
- net NRST: track 74.3 -> 76.4 mm
- net GND: track 116.4 -> 118.4 mm, vias 59 -> 61
- net /QON: track 44.9 -> 46.1 mm
