File: pcb/resonance_converter_controller_io/resonance_converter_controller_io.kicad_sch (KiCad schematic)
At the start: 53 parts, among them J1 DF12NB_5.0_-20DP-0.5V_51_, J2 Conn_01x30_MountingPin, J3 Conn_01x02, J4 Conn_01x02, J7 Conn_ARM_SWD_TagConnect_TC2030, SW1 RotaryEncoder_Switch_MP, SW2 SW_SPST, SW3 SW_SPST, SW4 SW_SPST, SW5 SW_SPST, U1 PCF8574RGTR, U2 TLV61047DDC, U3 AXK6S40647YG

Commit message: Update pcb
Parts:
- added C19, C20: 100nF, Capacitor_SMD:C_0402_1005Metric, symbol Device:C
Connections:
- net GND: now also C19.2, C20.2
- net NRST: now also C19.1
- net VOUT: now also U3.21, U3.23, U3.25, U3.27, U3.29, U3.31, U3.33, U3.35, U3.37, U3.39; no longer U3.22, U3.24, U3.26, U3.28, U3.30, U3.32, U3.34, U3.36, U3.38, U3.40
- net VSYS: now also U3.22, U3.24, U3.26, U3.28, U3.30, U3.32, U3.34, U3.36, U3.38, U3.40; no longer U3.21, U3.23, U3.25, U3.27, U3.29, U3.31, U3.33, U3.35, U3.37, U3.39
- net /QON: now also C20.1
